File: tests/fixtures/switch_project/switch.kicad_pcb (KiCad board)
At the start: 2 copper layers, 40 x 15 mm, 2 parts

Commit message: examples/jlcpcb: JLCPCB Gerber export tooling + corrected design rules
Captured for dev purposes — adjacent to the core KliCAD fork, not
central to it, but worth preserving in version control.

  - export_jlcpcb.py: the JLCPCB Gerber + drill export "algorithm",
    reproducing JLCPCB's official KiCad-9 help-article procedure.
    Drives a running KliCAD instance: loads the board, runs DRC
    (aborts on errors), exports Gerbers (Protel extensions, X2
    format, netlist attributes, edge-on-all-layers, zone-fill check)
    and drill (Excellon, absolute, mm, decimal, alternate oval,
    PTH+NPTH merged), then zips for upload.  Builds the layer list
    from the board's copper-layer count so it handles multilayer too.

  - JLCPCB_2layer.kicad_dru: corrected JLCPCB design-rule set,
    cross-checked against jlcpcb.com/capabilities.  Fixes the two
    errors found across the community .kicad_dru lineage (darkxst ->
    denniskupec -> labtroll -> EddyBeaupre): the dangerous 0.075mm
    annular ring (official: 0.20mm) and the systemic 0.127mm SMD
    pad-to-pad under-spec (official: 0.15mm).

  - README.md: documents the rule-file lineage audit + the export
    settings + the export-binding getBoard() footgun the script
    works around.

Also commits the switch fixture board edits (back-side silkscreen +
mirrored "2026" date text) made while validating the export end to
end against JLCPCB rules.

Co-Authored-By: Claude Opus 4.7 (1M context) <noreply@anthropic.com>
Other:
- board text added: "2026"
- board text added: "RFC.US"
Changed lines of the file:
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@@
 		(layer "Edge.Cuts")
+	)
+	(gr_text "RFC.US"
+		(at 127.5 88.6 0)
+		(layer "B.SilkS")
+		(effects
+			(font
+				(size 1.5 1.5)
+				(thickness 0.3)
+				(bold yes)
+			)
+			(justify left bottom mirror)
+		)
+	)
+	(gr_text "2026"
+		(at 154.7 88.6 0)
+		(layer "B.SilkS")
+		(effects
+			(font
+				(size 1.5 1.5)
+				(thickness 0.3)
+				(bold yes)
+			)
+			(justify left bottom mirror)
+		)
 	)
 	(segment
